File: hardware/eagle/AutomatonXL320/AutomatonXL320.sch (EAGLE design)
At the start: 46 parts, among them J1 USB_RCPT_10118192-0001LF, J2 ESP_ROBOT_BOARD_GPIO_16, J6 BATTERY, U1 ESP-WROOM-32D, U2 CP2102N-A02-GQFN20, U3 TPS62143RGTT, U4 TXB0106PWRPW16-L, U5 NC7WZ241K8X, U7 TPS62056DGSRDGS10-M

Commit message: CP2102N VBUS is now connected via resistor ladder
* CP2102N was overheating at times because it was
  connected directly to USB VBUS
Parts:
- added R10: 22.1k, TimeExpander2:RESISTOR0402
- added R11: 47.5k, TimeExpander2:RESISTOR0402
- R1, R2, R3, R5, R8, R9: value 10k -> RESISTOR0402; device TimeExpander2:RESISTOR -> TimeExpander2:RESISTOR0402
- R15: value 130k -> RESISTOR0402; device TimeExpander2:RESISTOR -> TimeExpander2:RESISTOR0402
- R16, R4: value 100k -> RESISTOR0402; device TimeExpander2:RESISTOR -> TimeExpander2:RESISTOR0402
- R17, R18: value 1M -> RESISTOR0402; device TimeExpander2:RESISTOR -> TimeExpander2:RESISTOR0402
- R7: value 1k -> RESISTOR0402; device TimeExpander2:RESISTOR -> TimeExpander2:RESISTOR0402
Connections:
- new net N$18: R10.P$2, R11.P$1, U2A.VBUS
- net GND: now also R11.P$2
- net N$15: now also R10.P$1; no longer U2A.VBUS
Other:
- moved on the sheet: J1
